Commit message: recover collision for 9 joints, still work

File: resources/robots/go1/urdf/go1.urdf (robot description, URDF)
Before this commit: robot go1_description, 38 links, 37 joints
Links:
- link FL_hip: geometry collision cylinder length=0.04 radius=0.046; visual mesh filename=../meshes/hip.dae scale=1 1 1
- link FL_thigh_shoulder: geometry collision cylinder length=0.032 radius=0.041
- link FR_hip: geometry collision cylinder length=0.04 radius=0.046; visual mesh filename=../meshes/hip.dae scale=1 1 1
- link FR_thigh_shoulder: geometry collision cylinder length=0.032 radius=0.041
- link RL_hip: geometry collision cylinder length=0.04 radius=0.046; visual mesh filename=../meshes/hip.dae scale=1 1 1
- link RL_thigh_shoulder: geometry collision cylinder length=0.032 radius=0.041
- link RR_hip: geometry collision cylinder length=0.04 radius=0.046; visual mesh filename=../meshes/hip.dae scale=1 1 1
- link RR_thigh_shoulder: geometry collision cylinder length=0.032 radius=0.041
- link imu_link: geometry collision box size=.001 .001 .001; visual box size=0.001 0.001 0.001
